File: 02.Hardware/MK2 PCBs/02.CONNECTORS/Connectors-MK2.brd (EAGLE design)
At the start: 59.5 x 28.5 mm, 20 parts, among them K1 FLEX8, Q1 310mA/60V/1.6Ω, Q2 310mA/60V/1.6Ω, Q3 310mA/60V/1.6Ω, Q4 310mA/60V/1.6Ω, Q5 310mA/60V/1.6Ω, Q6 SI4459ADY-T1-GE3, Q7 SI4459ADY-T1-GE3

Commit message: pequeños cambios ruteado
Routing:
- net VCC: track 69.1 -> 50.3 mm, vias 3 -> 4
- net VOUT: track 69.5 -> 80.5 mm
- net MACHINE_1: track 19.1 -> 28.2 mm
- net MACHINE_2: track 9.51 -> 16.5 mm
- net GND: track 83.5 -> 87.6 mm
- net N$5: track 10.0 -> 10.8 mm
Other:
- board text added: "somos la fucking puta ostia"
- board text removed: "fucking puta ostia"
