File: 02.Hardware/MK2 2040/01.EDCPSU/EDCPSUMK2_2040.brd (EAGLE design)
At the start: 96 x 60.8 mm, 174 parts, among them IC1 W25Q64JVSSIQ, IC2 74LVC1G74DP,125, J1 DX07S016JA1R1500, J2 RP2040TR7, J4 FTDI_DEVICE, J6 Display, K1 FLEX8, Q1 PJA3416AE_R1_00001, Q2 2N7002PW, Q4 2N7002PW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

Commit message: Propuesta 1 MK2 2040
Parts:
- removed C44: 100n, SparkFun:0805
- removed D1: SM2T18A, SM2T18A:SM2T18A
- removed IC2: 74LVC1G74DP,125, 74LVC1G74DP_125:SOP65P400X110-8N
- removed U8: TPS54531, EDCPSU - Rev3:SOIC8
- added BZ1: PKMCS0909E4000-R1, buzzer:PKMCS0909
- added C59, C61: 100n, SparkFun:0805
- added C60: 100n, rcl:C0805
- added D3: SMAJ24CA, SMAJ24CA:DIONM5127X229N
- added D4: PESD5V0U2BT,215, PESD5V0U2BT_215:SOT95P230X110-3N
- added D5: 3SMAJ5923B-TP, 3SMAJ5923B-TP:DIOM4325X244N
- added IC3: AP64501SP-13, AP64501SP-13:SOIC127P600X163-9N
- added L7: MMZ2012Y202BT000, SparkFun:0805
- added R40: 43K, SparkFun:0805
- added R45: 22K, SparkFun:0805
- added R46: 33, SparkFun:0805
- added R57: 10k, SparkFun:0805
- added R61: 330, SparkFun:0805
- added U1: MCP4725, SparkFun-IC-Conversion:SOT23-6
- C30: value 15n -> 33n
- C37: value 2.2n -> 10n
- C38: value 15p -> 16p
- D6: value Diode -> BAV199; device EDCPSU - Rev3:DO-214AB -> diode:SOT23
- R10: value 22K -> 91K
- R11: value 10K -> 10k
- R3: value 11K -> N.C.
- R4: value 5K6 -> N.C
- R44: value 33K -> 25k
- R5: value 2K8 -> 11K
- R6: value 1K4 -> 5K6
- R7: value 180K -> 2K8
- R8: value 91K -> 1K4
- R9: value 43K -> 180K
- moved D6 291.8 mm to (-19.8, -221.7)
- moved R3 255.4 mm to (-14.5, -199.3), turned to 0 degrees
- moved R9 241.6 mm to (-14.5, -185.6), turned to 0 degrees
- moved R10 240.7 mm to (-11.6, -185.6), turned to 0 degrees
- moved R5 239.0 mm to (-11.6, -182.4), turned to 0 degrees
- moved R7 238.8 mm to (-5.70, -182.4), turned to 0 degrees
- moved R6 238.7 mm to (-8.63, -182.4), turned to 0 degrees
- moved R8 237.9 mm to (-2.77, -182.4), turned to 0 degrees
- moved L6 232.8 mm to (-7.85, -179.1)
- moved L5 229.1 mm to (-14.5, -179.1)
- moved U7 224.4 mm to (-8.86, -174.2), turned to 0 degrees
- moved R4 217.4 mm to (-11.0, -160.8), turned to 0 degrees
Connections:
- removed net N$3: R5.1, U7.4
- removed net N$64: D1.2, LS1.2, Q1.3
- new net BUZZ: R46.1
- new net C_CC1: J1.3, R55.2
- new net C_CC2: J1.9, R56.2
- new net C_SBU1: J1.10
- new net C_SBU2: J1.4
- new net FB_DAC: R4.1, U1.1
- new net N$16: R45.1, U7.11
- new net N$19: D5.A, OP1.1
- new net N$66: BZ1.2, D6.3, LS1.2, Q1.3, R61.1
- new net N$68: BZ1.1, C61.2, D6.2, L7.2, LS1.3, R61.2
- new net SCL1: L5.2
- new net USB_D+: D4.2, J1.6, J1.7
- new net USB_D-: D4.1, J1.5, J1.8
- net CC1: no longer J1.3, R55.2
- net CC2: no longer J1.9, R56.2
- net EN_TPS54531: now also IC3.3; no longer U8.3
- net GND: now also C59.1, C60.1, C61.1, D3.1, D4.3, IC3.7, IC3.9, R3.1, R57.2, U1.2, U1.6; no longer C44.1, D6.1, U8.7, U8.PAD
- net IN+: now also D3.2
- net N$1: now also R5.1; no longer R3.1
- net N$2: now also R6.1; no longer R4.1
- net N$4: now also R7.1, U7.4; no longer R6.1, U7.3
- net N$44: now also IC3.4; no longer U8.4
- net N$47: now also IC3.1; no longer U8.1
- net N$48: now also IC3.5, R40.2, R45.2; no longer U8.5
- net N$5: now also R8.1, U7.3; no longer R7.1, U7.14
- net N$51: now also IC3.8; no longer D6.2, U8.8
- net N$52: now also IC3.6; no longer U8.6
- net N$65: now also R46.2, R57.1
- net N$7: now also R9.1, U7.14; no longer R8.1, U7.13
- net N$8: now also R10.1, U7.13; no longer R9.1, U7.12
- net N$9: now also R40.1, U7.12; no longer R10.1, U7.11
- net SCL: now also U1.5; no longer L5.2
- net SDA: now also U1.4
- net VCC: now also C60.2, D5.C, IC3.2, L7.1, U1.3; no longer OP1.1, U8.2
- net VCC-ISO: now also C59.2; no longer C44.2, D1.1, LS1.3
Routing:
- net VCC: track 83.7 -> 32.3 mm, vias 8 -> 6
- net GND: track 163.4 -> 133.2 mm, vias 142 -> 141
- net N$9: track 19.6 -> 0.00 mm
- net N$48: track 20.5 -> 1.76 mm
- net N$5: track 14.8 -> 0.00 mm, vias 2 -> 0
- net N$8: track 13.6 -> 0.00 mm
- net N$7: track 12.7 -> 0.00 mm, vias 2 -> 0
- net VCC-ISO: track 82.3 -> 71.4 mm, vias 13 -> 12
- net N$40: track 7.91 -> 0.00 mm, vias 2 -> 0
- net N$51: track 25.9 -> 20.5 mm
- net N$54: track 4.88 -> 0.00 mm
- net N$4: track 3.18 -> 0.00 mm
- net IN+: track 31.3 -> 28.3 mm, vias 8 -> 6
- net N$3: track 2.71 -> 0.00 mm
- net N$2: track 2.48 -> 0.00 mm
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
Commit message: Version de comienzo de rediseño
Parts:
- added C44: 10uF, SparkFun-Passives:1206
- added C62: 22u 10V X5R, SparkFun:0805
- added C63, C64: 4.7u 50V X5R, SparkFun:0805
- added R58: 330, SparkFun:0805
- C50: value 27p -> 22u 10V X5R
Connections:
- net OVC_ALARM renamed VIN_ALARM
- new net N$3: C44.1, D6.2, LS1.3
- new net VISENSE: R30.1
- net GND: now also C44.2, C62.1, C63.1, C64.1, R58.2
- net IN_OVC: no longer R30.1
- net N$14: now also R58.1
- net N$68: no longer D6.2, LS1.3
- net VCC: now also C63.2, C64.2
- net VCC-ISO: now also C62.2
Routing:
- net IN_OVC: track 98.2 -> 97.0 mm
Changed lines of the file:
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@@
 <drawing>
 <settings>
-<setting alwaysvectorfont="yes"/>
+<setting alwaysvectorfont="no"/>
 <setting keepoldvectorfont="yes"/>
 <setting verticaltext="up"/>
@@
 <attribute name="VALUE" x="1.814" y="-118.117" size="0.4064" layer="27"/>
 </element>
-<element name="C50" library="SparkFun" package="0805" value="27p" x="2.83" y="-120" smashed="yes">
+<element name="C50" library="SparkFun" package="0805" value="22u 10V X5R" x="2.83" y="-120" smashed="yes">
 <attribute name="NAME" x="2.068" y="-119.1745" size="0.4064" layer="25"/>
 <attribute name="VALUE" x="1.814" y="-121.397" size="0.4064" layer="27"/>
@@
 <attribute name="VALUE" x="-18.84" y="-238.54" size="1.27" layer="27"/>
 </element>
+<element name="C44" library="SparkFun-Passives" package="1206" value="10uF" x="-19.75" y="-247.86" smashed="yes">
+<attribute name="NAME" x="-21.02" y="-246.717" size="0.4064" layer="25"/>
+<attribute name="VALUE" x="-21.147" y="-249.384" size="0.4064" layer="27"/>
+</element>
+<element name="R58" library="SparkFun" package="0805" value="330" x="-23.67" y="-247.98" smashed="yes">
+<attribute name="NAME" x="-24.432" y="-247.1545" size="0.4064" layer="25"/>
+<attribute name="VALUE" x="-24.686" y="-249.377" size="0.4064" layer="27"/>
+</element>
+<element name="C62" library="SparkFun" package="0805" value="22u 10V X5R" x="-26.62" y="-247.98" smashed="yes">
+<attribute name="NAME" x="-27.382" y="-247.1545" size="0.4064" layer="25"/>
+<attribute name="VALUE" x="-27.636" y="-249.377" size="0.4064" layer="27"/>
+</element>
+<element name="C63" library="SparkFun" package="0805" value="4.7u 50V X5R" x="-29.57" y="-247.98" smashed="yes">
+<attribute name="NAME" x="-30.332" y="-247.1545" size="0.4064" layer="25"/>
+<attribute name="VALUE" x="-30.586" y="-249.377" size="0.4064" layer="27"/>
+</element>
+<element name="C64" library="SparkFun" package="0805" value="4.7u 50V X5R" x="-32.52" y="-247.98" smashed="yes">
+<attribute name="NAME" x="-33.282" y="-247.1545" size="0.4064" layer="25"/>
+<attribute name="VALUE" x="-33.536" y="-249.377" size="0.4064" layer="27"/>
+</element>
 </elements>
 <signals>
@@
 <contactref element="C61" pad="1"/>
 <contactref element="R57" pad="2"/>
+<contactref element="C44" pad="2"/>
+<contactref element="R58" pad="2"/>
+<contactref element="C62" pad="1"/>
+<contactref element="C63" pad="1"/>
+<contactref element="C64" pad="1"/>
 <wire x1="-3.67" y1="-240.42" x2="-11.33" y2="-240.42" width="0" layer="19" extent="1-1"/>
+<wire x1="-18.35" y1="-247.86" x2="-11.33" y2="-240.42" width="0" layer="19" extent="1-1"/>
+<wire x1="-22.77" y1="-247.98" x2="-18.35" y2="-247.86" width="0" layer="19" extent="1-1"/>
+<wire x1="-27.52" y1="-247.98" x2="-22.77" y2="-247.98" width="0" layer="19" extent="1-1"/>
+<wire x1="-30.47" y1="-247.98" x2="-27.52" y2="-247.98" width="0" layer="19" extent="1-1"/>
+<wire x1="-33.42" y1="-247.98" x2="-30.47" y2="-247.98" width="0" layer="19" extent="1-1"/>
 <wire x1="-12.14" y1="-206.3" x2="-11.33" y2="-240.42" width="0" layer="19" extent="1-1"/>
 <wire x1="-14.13" y1="-202.85" x2="-12.14" y2="-206.3" width="0" layer="19" extent="1-1"/>
@@
 <contactref element="D5" pad="C"/>
 <contactref element="L7" pad="1"/>
+<contactref element="C63" pad="2"/>
+<contactref element="C64" pad="2"/>
 <wire x1="-13.92" y1="-194.4299" x2="-20.135" y2="-214.68" width="0" layer="19" extent="1-1"/>
 <wire x1="-13.07" y1="-190.51" x2="-13.92" y2="-194.4299" width="0" layer="19" extent="1-1"/>
 <wire x1="-17.97" y1="-240.42" x2="-20.135" y2="-214.68" width="0" layer="19" extent="1-1"/>
+<wire x1="-28.67" y1="-247.98" x2="-17.97" y2="-240.42" width="0" layer="19" extent="1-1"/>
+<wire x1="-31.62" y1="-247.98" x2="-28.67" y2="-247.98" width="0" layer="19" extent="1-1"/>
 <wire x1="-7.78" y1="-152.735" x2="-13.07" y2="-190.51" width="0" layer="19" extent="1-1"/>
 <wire x1="6.86" y1="-111.24" x2="-7.78" y2="-152.735" width="0" layer="19" extent="1-1"/>
@@
 <contactref element="C59" pad="2"/>
 <contactref element="U7" pad="1"/>
+<contactref element="C62" pad="2"/>
 <wire x1="-13.305" y1="-177.01" x2="-13.59" y2="-182.36" width="0" layer="19" extent="1-1"/>
 <wire x1="6.64" y1="-134.8" x2="-13.305" y2="-177.01" width="0" layer="19" extent="1-1"/>
@@
 <wire x1="104.2206" y1="31.0413" x2="95.1" y2="29.294" width="0" layer="19" extent="16-16"/>
 <wire x1="108.68" y1="41.86" x2="104.2206" y2="31.0413" width="0" layer="19" extent="1-16"/>
+<wire x1="-25.72" y1="-247.98" x2="-13.59" y2="-182.36" width="0" layer="19" extent="1-1"/>
 </signal>
 <signal name="RX-I">
@@
 </polygon>
 </signal>
-<signal name="OVC_ALARM">
+<signal name="VIN_ALARM">
 <contactref element="U6" pad="10"/>
 <contactref element="TP10" pad="1"/>
@@
 <wire x1="23.495" y1="27.33" x2="22.395" y2="26.23" width="0.4064" layer="1"/>
 <wire x1="21.495" y1="26.23" x2="22.395" y2="26.23" width="0.4064" layer="1"/>
-<contactref element="R30" pad="1"/>
 <wire x1="33.656709375" y1="41.918290625" x2="34.63841875" y2="42.9" width="0.254" layer="2"/>
 <wire x1="34.63841875" y1="42.9" x2="53.145" y2="42.9" width="0.254" layer="2"/>
@@
 <wire x1="83.65" y1="45.97" x2="82.3668" y2="47.2532" width="0.254" layer="1"/>
 <wire x1="83.65" y1="44.138" x2="83.65" y2="45.97" width="0.254" layer="1"/>
-<wire x1="82.755" y1="56.56" x2="81.605" y2="56.56" width="0.254" layer="1"/>
 </signal>
 <signal name="N$14">
@@
 <wire x1="79.805" y1="54.845" x2="79.805" y2="56.56" width="0.4064" layer="1"/>
 <wire x1="79.412" y1="54.452" x2="79.805" y2="54.845" width="0.4064" layer="1"/>
+<contactref element="R58" pad="1"/>
+<wire x1="-24.57" y1="-247.98" x2="78.585" y2="54.452" width="0" layer="19" extent="1-1"/>
 </signal>
 <signal name="SPARE2">
@@
 <contactref element="C61" pad="2"/>
 <contactref element="BZ1" pad="1"/>
-<contactref element="LS1" pad="3"/>
-<contactref element="D6" pad="2"/>
-<wire x1="-18.88" y1="-222.76" x2="-20.84" y2="-232.04" width="0" layer="19" extent="1-1"/>
 <wire x1="-16.17" y1="-240.42" x2="-20.84" y2="-232.04" width="0" layer="19" extent="1-1"/>
 <wire x1="-19.82" y1="-244.22" x2="-16.17" y2="-240.42" width="0" layer="19" extent="1-1"/>
 <wire x1="-9.53" y1="-240.42" x2="-16.17" y2="-240.42" width="0" layer="19" extent="1-1"/>
+</signal>
+<signal name="N$3">
+<contactref element="LS1" pad="3"/>
+<contactref element="D6" pad="2"/>
+<contactref element="C44" pad="1"/>
+<wire x1="-21.15" y1="-247.86" x2="-18.88" y2="-222.76" width="0" layer="19" extent="1-1"/>
 <wire x1="9.71" y1="-77" x2="-18.88" y2="-222.76" width="0" layer="19" extent="1-1"/>
 </signal>
+<signal name="VISENSE">
+<contactref element="R30" pad="1"/>
+</signal>
 </signals>
