File: 02.Hardware/MK2 2040/01.EDCPSU/EDCPSUMK2_2040.sch (EAGLE design)
At the start: 174 parts, among them IC1 W25Q64JVSSIQ, IC2 74LVC1G74DP,125, J1 DX07S016JA1R1500, J2 RP2040TR7, J4 FTDI_DEVICE, J6 Display, K1 FLEX8, Q1 PJA3416AE_R1_00001, Q2 2N7002PW, Q4 2N7002PW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

Commit message: Propuesta 1 MK2 2040
Parts:
- removed C44: 100n, SparkFun:CAP0805
- removed D1: SM2T18A, SM2T18A:SM2T18A
- removed IC2: 74LVC1G74DP,125, 74LVC1G74DP_125:74LVC1G74DP,125
- removed U8: TPS54531, EDCPSU - Rev3:TPS5431DDAR
- added BZ1: PKMCS0909E4000-R1, buzzer:PKMCS0909E4000-R1
- added C59, C61: 100n, SparkFun:CAP0805
- added C60: 100n, rcl:C-EUC0805
- added D3: SMAJ24CA, SMAJ24CA:SMAJ24CA
- added D4: PESD5V0U2BT,215, PESD5V0U2BT_215:PESD5V0U2BT,215
- added D5: 3SMAJ5923B-TP, 3SMAJ5923B-TP:3SMAJ5923B-TP
- added IC3: AP64501SP-13, AP64501SP-13:AP64501SP-13
- added L7: MMZ2012Y202BT000, SparkFun:RESISTOR0805-RES
- added R40: 43K, SparkFun:RESISTOR0805-RES
- added R45: 22K, SparkFun:RESISTOR0805-RES
- added R46: 33, SparkFun:RESISTOR0805-RES
- added R57: 10k, SparkFun:RESISTOR0805-RES
- added R61: 330, SparkFun:RESISTOR0805-RES
- added U1: MCP4725, SparkFun-IC-Conversion:MCP4725SOT-23
- C30: value 15n -> 33n
- C37: value 2.2n -> 10n
- C38: value 15p -> 16p
- D6: value Diode -> BAV199; device EDCPSU - Rev3:DSMC -> diode:BAV199
- R10: value 22K -> 91K
- R11: value 10K -> 10k
- R3: value 11K -> N.C.
- R4: value 5K6 -> N.C
- R44: value 33K -> 25k
- R5: value 2K8 -> 11K
- R6: value 1K4 -> 5K6
- R7: value 180K -> 2K8
- R8: value 91K -> 1K4
- R9: value 43K -> 180K
Connections:
- removed net N$3: R5.1, U7.DRAIN1
- removed net N$64: D1.A, LS1.-, Q1.D
- new net BUZZ: R46.1
- new net C_CC1: J1.CC1, R55.2
- new net C_CC2: J1.CC2, R56.2
- new net C_SBU1: J1.SBU1
- new net C_SBU2: J1.SBU2
- new net FB_DAC: R4.1, U1.VOUT
- new net N$16: R45.1, U7.DRAIN4
- new net N$19: D5.A, OP1.A
- new net N$66: BZ1.-, D6.AC, LS1.-, Q1.D, R61.1
- new net N$68: BZ1.+, C61.2, D6.C, L7.2, LS1.DUMMY, R61.2
- new net SCL1: L5.2
- new net USB_D+: D4.CATHODE_2, J1.D+
- new net USB_D-: D4.CATHODE_1, J1.D-
- net CC1: no longer J1.CC1, R55.2
- net CC2: no longer J1.CC2, R56.2
- net EN_TPS54531: now also IC3.EN; no longer U8.EN
- net GND: now also C59.1, C60.1, C61.1, D3.1, D4.COMMON_CATHODE, IC3.EP, IC3.GND, R3.1, R57.2, U1.AO, U1.VSS; no longer C44.1, D6.A, U8.GND, U8.PAD
- net IN+: now also D3.2
- net N$1: now also R5.1; no longer R3.1
- net N$2: now also R6.1; no longer R4.1
- net N$4: now also R7.1, U7.DRAIN1; no longer R6.1, U7.DRAIN0
- net N$44: now also IC3.SS; no longer U8.SS
- net N$47: now also IC3.BST; no longer U8.BOOT
- net N$48: now also IC3.FB, R40.2, R45.2; no longer U8.VSENSE
- net N$5: now also R8.1, U7.DRAIN0; no longer R7.1, U7.DRAIN7
- net N$51: now also IC3.SW; no longer D6.K, U8.PH
- net N$52: now also IC3.COMP; no longer U8.COMP
- net N$65: now also R46.2, R57.1
- net N$7: now also R9.1, U7.DRAIN7; no longer R8.1, U7.DRAIN6
- net N$8: now also R10.1, U7.DRAIN6; no longer R9.1, U7.DRAIN5
- net N$9: now also R40.1, U7.DRAIN5; no longer R10.1, U7.DRAIN4
- net SCL: now also U1.SCL; no longer L5.2
- net SDA: now also U1.SDA
- net VCC: now also C60.2, D5.K, IC3.VIN, L7.1, U1.VDD; no longer OP1.A, U8.VIN
- net VCC-ISO: now also C59.2; no longer C44.2, D1.K, LS1.DUMMY
Other:
- note removed: "COMPARATOR"
- note removed: "Puerto Serie"
- moved on the sheet: C19, C20, C35, C36, C38, C53, C55, C57, IN-, J1, L5, L6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

Commit message: Version de comienzo de rediseño
Parts:
- added C44: 10uF, SparkFun-Passives:CAP1206
- added C62: 22u 10V X5R, SparkFun:CAP0805
- added C63, C64: 4.7u 50V X5R, SparkFun:CAP0805
- added R58: 330, SparkFun:RESISTOR0805-RES
- C50: value 27p -> 22u 10V X5R
Connections:
- net OVC_ALARM renamed VIN_ALARM
- new net N$3: C44.1, D6.C, LS1.DUMMY
- new net VISENSE: R30.1
- net GND: now also C44.2, C62.1, C63.1, C64.1, R58.2
- net IN_OVC: no longer R30.1
- net N$14: now also R58.1
- net N$68: no longer D6.C, LS1.DUMMY
- net VCC: now also C63.2, C64.2
- net VCC-ISO: now also C62.2
Other:
- note added: "ADC reference Usar esta referencia de DIGIKEY (SOT-23) LM4040C25FTA"
- note added: "Añadir diodo zener de 3v6 en paralelo con la salida (C50) Usar SOD-123 referencia Digikey: MMSZ5227B-TP"
- note added: "Cambiar este integrado en la BOM por este equivalente: SN74AC14PWR Ojo! pq este TSSOP-14 es 1mm mas estrecho que el original"
- note added: "Dejar espacio para el DIODO. No quitar para poder aprovechar las 500 uds. que tiene SETI"
- note added: "Diodo zener de 8V2 añadido Este diodo tiene que llevar una buena disipación pq se lleva 125mW cdo el pedal esta activado"
- note added: "El transistor el que había 2N7002W"
- note added: "Hay que mirar si el de 25V que va en el DCDC tiene un precio razonable como para no buscar otro distinto en 10uF / 6V"
- note added: "Indicar esta referencia en el part number TLRP3A30CR050FTE"
- note added: "Nuevo. Susituye al diodo que habia antes"
- note added: "OJO: Indicar en el esquematico que es el AP63203 !!"
- note added: "Sensado del voltaje de entrada. Detección de caída por debajo de un nivel"
- note added: "VIN ALARM"
- note added: "a 3v3"
- note added: "cambiar D8 por un TVS de 18v bidireccional con encapsulado: SMA (DO-214A)"
- note added: "comprueba si 1206 (que es lo que tienes puesto) es el valor más típico (y barato) en 10uF /25V Tambien indica lo de los 25V en el valor para que quede claro"
- note removed: "Falta: - ADC reference"
- note removed: "OVC ALARM"
- moved on the sheet: BZ1, C61, D6, L7, LS1, Q1, R30, R46, R57, R61
