File: 02.Hardware/MK2 2040/05. TESTER RP2040/tester rp2040.brd (EAGLE design)
At the start: 135 x 56 mm, 59 parts, among them IC1 MAX4634EUB+T, J1 302-S201, Q1 PJA3416AE_R1_00001, Q2 2N7002PW, Q3 2N7002PW, Q4 RQ3G110ATTB, Q5 PJA3416AE_R1_00001, Q6 2N7002PW, Q7 RQ3G110ATTB, Q8 PJA3416AE_R1_00001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

Commit message: Tester RP2040
Parts:
- added Z2, Z3: MMSZ5227B-7-F, MMSZ5227B-7-F:SOD3716X135N
Connections:
- new net N$2: Z1.2, Z3.2
- net IN+: now also Z2.1, Z2.2, Z3.1; no longer Z1.2
Changed lines of the file:
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@@
 <attribute name="VALUE" x="144.669" y="18.61" size="0.6096" layer="27" font="vector" ratio="20" rot="R90" align="top-center"/>
+</element>
+<element name="Z2" library="MMSZ5227B-7-F" package="SOD3716X135N" value="MMSZ5227B-7-F" x="25.9" y="1.6" smashed="yes">
+<attribute name="ARROW_PART_NUMBER" value="MMSZ5227B-7-F" x="22.35" y="1.6" size="1.778" layer="27" display="off"/>
+<attribute name="ARROW_PRICE-STOCK" value="https://www.arrow.com/en/products/mmsz5227b-7-f/diodes-incorporated" x="22.35" y="1.6" size="1.778" layer="27" display="off"/>
+<attribute name="DESCRIPTION" value="Diode Zener 3.6V 5% 500mW 2Pin SOD123 Diodes Inc MMSZ5227B-7-F Zener Diode, 3.6V 5% 500 mW SMT 2-Pin SOD-123" x="22.35" y="1.6" size="1.778" layer="27" display="off"/>
+<attribute name="HEIGHT" value="1.35mm" x="22.35" y="1.6" size="1.778" layer="27" display="off"/>
+<attribute name="MANUFACTURER_NAME" value="Diodes Inc." x="22.35" y="1.6" size="1.778" layer="27" display="off"/>
+<attribute name="MANUFACTURER_PART_NUMBER" value="MMSZ5227B-7-F" x="22.35" y="1.6" size="1.778" layer="27" display="off"/>
+<attribute name="MOUSER_PART_NUMBER" value="621-MMSZ5227B-F" x="22.35" y="1.6" size="1.778" layer="27" display="off"/>
+<attribute name="MOUSER_PRICE-STOCK" value="https://www.mouser.com/Search/Refine.aspx?Keyword=621-MMSZ5227B-F" x="22.35" y="1.6" size="1.778" layer="27" display="off"/>
+<attribute name="NAME" x="25.9" y="1.6" size="1.27" layer="25" align="center"/>
+<attribute name="VALUE" x="25.9" y="1.6" size="1.27" layer="27" align="center"/>
+</element>
+<element name="Z3" library="MMSZ5227B-7-F" package="SOD3716X135N" value="MMSZ5227B-7-F" x="25.9" y="-1.8" smashed="yes">
+<attribute name="ARROW_PART_NUMBER" value="MMSZ5227B-7-F" x="22.4" y="-1.8" size="1.778" layer="27" display="off"/>
+<attribute name="ARROW_PRICE-STOCK" value="https://www.arrow.com/en/products/mmsz5227b-7-f/diodes-incorporated" x="22.4" y="-1.8" size="1.778" layer="27" display="off"/>
+<attribute name="DESCRIPTION" value="Diode Zener 3.6V 5% 500mW 2Pin SOD123 Diodes Inc MMSZ5227B-7-F Zener Diode, 3.6V 5% 500 mW SMT 2-Pin SOD-123" x="22.4" y="-1.8" size="1.778" layer="27" display="off"/>
+<attribute name="HEIGHT" value="1.35mm" x="22.4" y="-1.8" size="1.778" layer="27" display="off"/>
+<attribute name="MANUFACTURER_NAME" value="Diodes Inc." x="22.4" y="-1.8" size="1.778" layer="27" display="off"/>
+<attribute name="MANUFACTURER_PART_NUMBER" value="MMSZ5227B-7-F" x="22.4" y="-1.8" size="1.778" layer="27" display="off"/>
+<attribute name="MOUSER_PART_NUMBER" value="621-MMSZ5227B-F" x="22.4" y="-1.8" size="1.778" layer="27" display="off"/>
+<attribute name="MOUSER_PRICE-STOCK" value="https://www.mouser.com/Search/Refine.aspx?Keyword=621-MMSZ5227B-F" x="22.4" y="-1.8" size="1.778" layer="27" display="off"/>
+<attribute name="NAME" x="25.9" y="-1.8" size="1.27" layer="25" align="center"/>
+<attribute name="VALUE" x="25.9" y="-1.8" size="1.27" layer="27" align="center"/>
 </element>
 </elements>
@@
 <contactref element="Q7" pad="8"/>
 <contactref element="Q7" pad="5"/>
-<contactref element="Z1" pad="2"/>
 <wire x1="31.22" y1="28.06" x2="35.96" y2="28.06" width="1.016" layer="16"/>
 <wire x1="78.1" y1="41.95" x2="78.2" y2="41.85" width="1.016" layer="16"/>
@@
 <via x="78.3" y="43.1" extent="1-16" drill="0.35"/>
 <via x="79.2" y="41.7" extent="1-16" drill="0.35"/>
+<contactref element="Z2" pad="2"/>
+<contactref element="Z2" pad="1"/>
+<contactref element="Z3" pad="1"/>
+<wire x1="81.7" y1="47.9" x2="81.8" y2="46.1" width="0" layer="19" extent="1-1"/>
+<wire x1="80.1" y1="47.6" x2="81.7" y2="47.9" width="0" layer="19" extent="1-1"/>
+<wire x1="79.4" y1="46.2" x2="80.1" y2="47.6" width="0" layer="19" extent="1-1"/>
+<wire x1="78.075" y1="47.915" x2="80.1" y2="47.6" width="0" layer="19" extent="1-1"/>
+<wire x1="78.2" y1="41.85" x2="78.2" y2="41.85" width="0" layer="19" extent="1-16"/>
+<wire x1="79.2" y1="41.7" x2="78.2" y2="41.85" width="0" layer="19" extent="1-1"/>
+<wire x1="78.3" y1="43.1" x2="78.2" y2="41.85" width="0" layer="19" extent="1-1"/>
+<wire x1="76.8" y1="41.1" x2="78.2" y2="41.85" width="0" layer="19" extent="1-1"/>
+<wire x1="76.9" y1="46.2" x2="76.775" y2="47.915" width="0" layer="19" extent="1-1"/>
+<wire x1="75.3" y1="46.4" x2="76.9" y2="46.2" width="0" layer="19" extent="1-1"/>
+<wire x1="80.9" y1="40.5" x2="79.2" y2="41.7" width="0" layer="19" extent="1-1"/>
+<wire x1="75.6" y1="42.9" x2="76.8" y2="41.1" width="0" layer="19" extent="1-1"/>
+<wire x1="80.9" y1="43.3" x2="79.2" y2="41.7" width="0" layer="19" extent="1-1"/>
+<wire x1="27.6" y1="1.6" x2="31.22" y2="28.06" width="0" layer="19" extent="1-1"/>
+<wire x1="24.2" y1="1.6" x2="27.6" y2="1.6" width="0" layer="19" extent="1-1"/>
+<wire x1="24.2" y1="-1.8" x2="24.2" y2="1.6" width="0" layer="19" extent="1-1"/>
 </signal>
 <signal name="VBUS_SENSE">
@@
 <wire x1="93.75" y1="36.35" x2="87.2" y2="29.8" width="0.508" layer="1"/>
 </signal>
+<signal name="N$2">
+<contactref element="Z1" pad="2"/>
+<contactref element="Z3" pad="2"/>
+<wire x1="27.6" y1="-1.8" x2="81.02" y2="41.85" width="0" layer="19" extent="1-1"/>
+</signal>
 </signals>
