File: 02.Hardware/MK2 2040/05. TESTER RP2040/tester rp2040.sch (EAGLE design)
At the start: 59 parts, among them IC1 MAX4634EUB+T, J1 302-S201, Q1 PJA3416AE_R1_00001, Q2 2N7002PW, Q3 2N7002PW, Q4 RQ3G110ATTB, Q5 PJA3416AE_R1_00001, Q6 2N7002PW, Q7 RQ3G110ATTB, Q8 PJA3416AE_R1_00001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

Commit message: Tester RP2040
Parts:
- added Z2, Z3: MMSZ5227B-7-F, MMSZ5227B-7-F:MMSZ5227B-7-F
Connections:
- new net N$2: Z1.A, Z3.A
- net IN+: now also Z2.A, Z2.K, Z3.K; no longer Z1.A
Other:
- moved on the sheet: Z1
Changed lines of the file:
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@@
 <part name="U$6" library="SparkFun-Aesthetics" deviceset="VCC-ISO" device="" value="3V3"/>
 <part name="U$7" library="SparkFun-Aesthetics" deviceset="VCC-ISO" device="" value="3V3"/>
+<part name="Z2" library="MMSZ5227B-7-F" deviceset="MMSZ5227B-7-F" device=""/>
+<part name="Z3" library="MMSZ5227B-7-F" deviceset="MMSZ5227B-7-F" device=""/>
 </parts>
 <sheets>
@@
 <attribute name="VALUE" x="173.99" y="93.98" size="1.778" layer="96" align="center-left"/>
 </instance>
-<instance part="Z1" gate="G$1" x="215.9" y="106.68" smashed="yes" rot="R90">
-<attribute name="NAME" x="220.98" y="115.57" size="1.778" layer="95" align="center-left"/>
-<attribute name="VALUE" x="220.98" y="113.03" size="1.778" layer="96" align="center-left"/>
+<instance part="Z1" gate="G$1" x="215.9" y="93.98" smashed="yes" rot="R90">
+<attribute name="NAME" x="220.98" y="102.87" size="1.778" layer="95" align="center-left"/>
+<attribute name="VALUE" x="220.98" y="100.33" size="1.778" layer="96" align="center-left"/>
 </instance>
 <instance part="Q5" gate="A" x="213.36" y="228.6" smashed="yes">
@@
 <instance part="U$7" gate="G$1" x="-116.84" y="38.1" smashed="yes" rot="MR0">
 <attribute name="VALUE" x="-115.824" y="41.656" size="1.778" layer="96" rot="MR0"/>
+</instance>
+<instance part="Z2" gate="G$1" x="205.74" y="160.02" smashed="yes" rot="R270">
+<attribute name="NAME" x="200.66" y="151.13" size="1.778" layer="95" rot="R180" align="center-left"/>
+<attribute name="VALUE" x="200.66" y="153.67" size="1.778" layer="96" rot="R180" align="center-left"/>
+</instance>
+<instance part="Z3" gate="G$1" x="226.06" y="160.02" smashed="yes" rot="R270">
+<attribute name="NAME" x="220.98" y="151.13" size="1.778" layer="95" rot="R180" align="center-left"/>
+<attribute name="VALUE" x="220.98" y="153.67" size="1.778" layer="96" rot="R180" align="center-left"/>
 </instance>
 </instances>
@@
 <wire x1="154.94" y1="127" x2="180.34" y2="127" width="0.1524" layer="91"/>
 <wire x1="180.34" y1="127" x2="180.34" y2="137.16" width="0.1524" layer="91"/>
-<wire x1="180.34" y1="144.78" x2="215.9" y2="144.78" width="0.1524" layer="91"/>
-<label x="243.84" y="144.78" size="1.27" layer="95" xref="yes"/>
-<pinref part="Z1" gate="G$1" pin="A"/>
-<wire x1="215.9" y1="144.78" x2="243.84" y2="144.78" width="0.1524" layer="91"/>
-<wire x1="215.9" y1="121.92" x2="215.9" y2="144.78" width="0.1524" layer="91"/>
-<junction x="215.9" y="144.78"/>
+<wire x1="180.34" y1="144.78" x2="205.74" y2="144.78" width="0.1524" layer="91"/>
 <junction x="180.34" y="137.16"/>
+<pinref part="Z2" gate="G$1" pin="A"/>
+</segment>
+<segment>
+<label x="243.84" y="160.02" size="1.27" layer="95" xref="yes"/>
+<wire x1="205.74" y1="160.02" x2="226.06" y2="160.02" width="0.1524" layer="91"/>
+<pinref part="Z2" gate="G$1" pin="K"/>
+<pinref part="Z3" gate="G$1" pin="K"/>
+<wire x1="226.06" y1="160.02" x2="243.84" y2="160.02" width="0.1524" layer="91"/>
+<junction x="226.06" y="160.02"/>
 </segment>
 </net>
@@
 <pinref part="Z1" gate="G$1" pin="K"/>
 <wire x1="177.8" y1="88.9" x2="215.9" y2="88.9" width="0.1524" layer="91"/>
-<wire x1="215.9" y1="88.9" x2="215.9" y2="106.68" width="0.1524" layer="91"/>
+<wire x1="215.9" y1="88.9" x2="215.9" y2="93.98" width="0.1524" layer="91"/>
 <junction x="177.8" y="81.28"/>
 </segment>
@@
 </segment>
 </net>
+<net name="N$2" class="0">
+<segment>
+<pinref part="Z1" gate="G$1" pin="A"/>
+<pinref part="Z3" gate="G$1" pin="A"/>
+<wire x1="215.9" y1="109.22" x2="226.06" y2="109.22" width="0.1524" layer="91"/>
+<wire x1="226.06" y1="109.22" x2="226.06" y2="144.78" width="0.1524" layer="91"/>
+</segment>
+</net>
